File: Hardware/PCB.brd (EAGLE design)
At the start: 170.2 x 111.2 mm, 103 parts, among them IC1 BD5229G-TR, IC4 XC6220A331MR-G, J1 FH34SRJ-24S-0.5SH_99_, J3 QWIIC_RIGHT_ANGLE, J4 112A-TAAR-R03_ATTEND, Q1 20V/4.2A/52mΩ/1.4W, Q2 20V/4.2A/52mΩ/1.4W, Q3 SI1308EDL-T1-GE3, U1 W25Q512JVEIQ, U2 ESP32-C6-WROOM-1-N8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

Commit message: add files
Parts:
- moved D12 4.38 mm to (12.7, 98.3)
- moved J4 4.10 mm to (5.86, 95.0)
- moved C9 3.81 mm to (10.4, 100.6)
- moved R8 3.19 mm to (6.66, 100.5)
Routing:
- net GND: track 731.2 -> 726.2 mm, vias 8 -> 10
- net MOSI: track 203.7 -> 208.0 mm
- net SCK: track 234.7 -> 238.0 mm
- net 3V3: track 479.0 -> 475.9 mm
- net SS_SD: track 99.3 -> 102.5 mm
- net MISO: track 132.8 -> 132.6 mm, vias 5 -> 7
Other:
- outline, holes or cut-outs redrawn

Commit message: add files"
Parts:
- moved C9 0.83 mm to (10.4, 101.4)
- moved D12 0.83 mm to (12.7, 99.2)
- moved J4 0.83 mm to (5.86, 95.9)
- moved R8 0.83 mm to (6.66, 101.3)
- moved C4_USB 0.15 mm to (157.6, 51.9)
- moved D1 0.15 mm to (154.7, 49.6)
- moved J2 0.15 mm to (167.3, 54.1)
- moved PFMF.050.1 0.15 mm to (154.8, 39.0)
- moved R2-USB 0.15 mm to (155.3, 44.6)
- moved R2-USB1 0.15 mm to (155.2, 46.4)
Routing:
- net MISO: track 132.6 -> 130.9 mm
- net MOSI: track 208.0 -> 209.3 mm
- net SS_SD: track 102.5 -> 103.5 mm
- net EPD_3V3: track 93.7 -> 92.9 mm
- net PREVGH: track 45.8 -> 45.3 mm
- net GND: track 726.2 -> 725.7 mm, vias 10 -> 57
- added copper zone on layer 1, net GND
- added copper zone on layer 16, net GND

Commit message: add files
Routing:
- net EPD_3V3_C: track 194.5 -> 191.0 mm
- net EPD_3V3: track 92.9 -> 94.4 mm
- net 32KHZ: track 97.0 -> 96.2 mm
- net SCK: track 238.0 -> 238.6 mm
- net GND: track 725.7 -> 726.0 mm, vias 57 -> 58
